File: Hardware/USB-C to TLL UART.kicad_pcb (KiCad board)
At the start: 2 copper layers, 26 x 30 mm, 13 parts, among them IC1 74LVC1G08SE-7, J1 Conn_01x06_Female, P1 USB_C_Plug_USB2.0, U1 CH340C, U2 AP2112K-3.3

Commit message: Updated Files
Parts:
- removed IC1: 74LVC1G08SE-7, SamacSys_Parts:SOT65P210X110-5N
- added TP1: TestPoint, TestPoint:TestPoint_Pad_1.5x1.5mm, F.Cu at (137.6, 89.0)
- added TP3: TestPoint, TestPoint:TestPoint_Pad_1.5x1.5mm, F.Cu at (148.9, 89.0)
- C1: value 10nF -> 0.1uF
- C2: value 100nF -> 10nF
- P1: footprint SnapEDA Library:GCT_USB4155-03-C_REVA -> Expansion_Card:USB_C_Plug_Molex_105444
- moved C1 11.8 mm to (132.5, 97.8), turned to 180 degrees
- moved C2 11.5 mm to (145.5, 98.8)
- moved C3 4.71 mm to (132.5, 99.0)
- moved P1 3.46 mm to (143.2, 90.0), turned to 0 degrees
- moved R1 3.41 mm to (139.8, 95.0)
- moved U1 1.37 mm to (143.5, 103.8)
- moved H2 0.62 mm to (154.8, 110.0)
- moved H1 0.43 mm to (131.7, 110.0)
- moved J1 0.16 mm to (141.5, 116.6)
Connections:
- C1 pad 1: Net-(C1-Pad1) -> 5V
- C2 pad 1: VCC -> Net-(C2-Pad1)
- U1 pad 1: Earth -> Net-(U1-Pad1)
- U1 pad 4: Net-(C1-Pad1) -> Net-(C2-Pad1)
Routing:
- net Earth: track 49.8 -> 21.6 mm, vias 3 -> 5
- net TXO: track 15.6 -> 33.0 mm, vias 1 -> 2
- net VCC: track 39.0 -> 23.7 mm
- net 5V: track 43.4 -> 48.6 mm, vias 1 -> 2
- net RXI: track 16.9 -> 21.1 mm, vias 0 -> 2
- net D-: track 9.23 -> 12.5 mm
- net Net-(C2-Pad1): track 0.00 -> 2.89 mm
- net Net-(C1-Pad1): track 2.72 -> 0.00 mm
- net D+: track 9.51 -> 12.0 mm, vias 1 -> 0
- net Net-(P1-PadA5): track 7.25 -> 5.89 mm, vias 2 -> 0
- net DTR: track 15.7 -> 14.9 mm, vias 1 -> 0
Other:
- outline, holes or cut-outs redrawn

Commit message: Updated files
Routing:
- net Earth: vias 5 -> 4
Changed lines of the file:
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@@
     (thickness 0.8)
     (drawings 33)
-    (tracks 107)
+    (tracks 106)
     (zones 0)
     (modules 14)
@@
     (36 B.SilkS user)
     (37 F.SilkS user)
-    (38 B.Mask user)
-    (39 F.Mask user)
+    (38 B.Mask user hide)
+    (39 F.Mask user hide)
     (40 Dwgs.User user hide)
     (41 Cmts.User user)
@@
   )
   (setup
-    (last_trace_width 0.3)
+    (last_trace_width 0.25)
     (user_trace_width 0.2)
     (user_trace_width 0.3)
@@
     (mod_text_size 1 1)
     (mod_text_width 0.15)
-    (pad_size 1.524 1.524)
-    (pad_drill 0.762)
+    (pad_size 0.3 1)
+    (pad_drill 0)
     (pad_to_mask_clearance 0)
     (aux_axis_origin 0 0)
@@
       (drillshape 0)
       (scaleselection 1)
-      (outputdirectory "C:/Users/Josh/Documents/ExpansionCards-main/Design Files/Complete Design Files/USB-C to TTL UART/SMD Assembly Files/"))
+      (outputdirectory "C:/Users/Josh/Documents/ExpansionCards-main/Design Files/Complete Design Files/USB-C to TTL UART/Gerbers/"))
   )
   (net 0 "")
@@
       (effects (font (size 1 1) (thickness 0.1)))
     )
-    (pad B12 smd rect (at -2.75 0.04) (size 0.38 1) (layers B.Cu B.Paste B.Mask)
-      (net 1 Earth))
-    (pad B11 smd rect (at -2.25 0.04) (size 0.38 1) (layers B.Cu B.Paste B.Mask))
-    (pad B10 smd rect (at -1.75 0.04) (size 0.38 1) (layers B.Cu B.Paste B.Mask))
-    (pad B9 smd rect (at -1.25 0.04) (size 0.38 1) (layers B.Cu B.Paste B.Mask)
-      (net 20 5V))
-    (pad B8 smd rect (at -0.75 0.04) (size 0.38 1) (layers B.Cu B.Paste B.Mask))
-    (pad B5 smd rect (at 0.75 0.04) (size 0.38 1) (layers B.Cu B.Paste B.Mask)
+    (pad B12 smd rect (at -2.75 0.04) (size 0.3 1) (layers B.Cu B.Paste B.Mask)
+      (net 1 Earth))
+    (pad B11 smd rect (at -2.25 0.04) (size 0.3 1) (layers B.Cu B.Paste B.Mask))
+    (pad B10 smd rect (at -1.75 0.04) (size 0.3 1) (layers B.Cu B.Paste B.Mask))
+    (pad B9 smd rect (at -1.25 0.04) (size 0.3 1) (layers B.Cu B.Paste B.Mask)
+      (net 20 5V))
+    (pad B8 smd rect (at -0.75 0.04) (size 0.3 1) (layers B.Cu B.Paste B.Mask))
+    (pad B5 smd rect (at 0.75 0.04) (size 0.3 1) (layers B.Cu B.Paste B.Mask)
       (net 5 "Net-(P1-PadB5)"))
-    (pad B4 smd rect (at 1.25 0.04) (size 0.38 1) (layers B.Cu B.Paste B.Mask)
-      (net 20 5V))
-    (pad B3 smd rect (at 1.75 0.04) (size 0.38 1) (layers B.Cu B.Paste B.Mask))
-    (pad B2 smd rect (at 2.25 0.04) (size 0.38 1) (layers B.Cu B.Paste B.Mask))
-    (pad B1 smd rect (at 2.75 0.04) (size 0.38 1) (layers B.Cu B.Paste B.Mask)
+    (pad B4 smd rect (at 1.25 0.04) (size 0.3 1) (layers B.Cu B.Paste B.Mask)
+      (net 20 5V))
+    (pad B3 smd rect (at 1.75 0.04) (size 0.3 1) (layers B.Cu B.Paste B.Mask))
+    (pad B2 smd rect (at 2.25 0.04) (size 0.3 1) (layers B.Cu B.Paste B.Mask))
+    (pad B1 smd rect (at 2.75 0.04) (size 0.3 1) (layers B.Cu B.Paste B.Mask)
       (net 1 Earth))
     (pad S1 smd rect (at 3.42 0.88) (size 0.7 1.15) (layers B.Cu B.Paste B.Mask)
@@
     (pad S1 smd rect (at -3.42 0.88) (size 0.7 1.15) (layers F.Cu F.Paste F.Mask)
       (net 1 Earth))
-    (pad A12 smd rect (at 2.75 0.04) (size 0.38 1) (layers F.Cu F.Paste F.Mask)
-      (net 1 Earth))
-    (pad A11 smd rect (at 2.25 0.04) (size 0.38 1) (layers F.Cu F.Paste F.Mask))
-    (pad A10 smd rect (at 1.75 0.04) (size 0.38 1) (layers F.Cu F.Paste F.Mask))
-    (pad A9 smd rect (at 1.25 0.04) (size 0.38 1) (layers F.Cu F.Paste F.Mask)
-      (net 20 5V))
-    (pad A8 smd rect (at 0.75 0.04) (size 0.38 1) (layers F.Cu F.Paste F.Mask))
-    (pad A7 smd rect (at 0.25 0.04) (size 0.38 1) (layers F.Cu F.Paste F.Mask)
+    (pad A12 smd rect (at 2.75 0.04) (size 0.3 1) (layers F.Cu F.Paste F.Mask)
+      (net 1 Earth))
+    (pad A11 smd rect (at 2.25 0.04) (size 0.3 1) (layers F.Cu F.Paste F.Mask))
+    (pad A10 smd rect (at 1.75 0.04) (size 0.3 1) (layers F.Cu F.Paste F.Mask))
+    (pad A9 smd rect (at 1.25 0.04) (size 0.3 1) (layers F.Cu F.Paste F.Mask)
+      (net 20 5V))
+    (pad A8 smd rect (at 0.75 0.04) (size 0.3 1) (layers F.Cu F.Paste F.Mask))
+    (pad A7 smd rect (at 0.25 0.04) (size 0.3 1) (layers F.Cu F.Paste F.Mask)
       (net 14 D-))
-    (pad A6 smd rect (at -0.25 0.04) (size 0.38 1) (layers F.Cu F.Paste F.Mask)
+    (pad A6 smd rect (at -0.25 0.04) (size 0.3 1) (layers F.Cu F.Paste F.Mask)
       (net 13 D+))
-    (pad A5 smd rect (at -0.75 0.04) (size 0.38 1) (layers F.Cu F.Paste F.Mask)
+    (pad A5 smd rect (at -0.75 0.04) (size 0.3 1) (layers F.Cu F.Paste F.Mask)
       (net 4 "Net-(P1-PadA5)"))
-    (pad A4 smd rect (at -1.25 0.04) (size 0.38 1) (layers F.Cu F.Paste F.Mask)
-      (net 20 5V))
-    (pad A3 smd rect (at -1.75 0.04) (size 0.38 1) (layers F.Cu F.Paste F.Mask))
-    (pad A2 smd rect (at -2.25 0.04) (size 0.38 1) (layers F.Cu F.Paste F.Mask))
-    (pad A1 smd rect (at -2.75 0.04) (size 0.38 1) (layers F.Cu F.Paste F.Mask)
+    (pad A4 smd rect (at -1.25 0.04) (size 0.3 1) (layers F.Cu F.Paste F.Mask)
+      (net 20 5V))
+    (pad A3 smd rect (at -1.75 0.04) (size 0.3 1) (layers F.Cu F.Paste F.Mask))
+    (pad A2 smd rect (at -2.25 0.04) (size 0.3 1) (layers F.Cu F.Paste F.Mask))
+    (pad A1 smd rect (at -2.75 0.04) (size 0.3 1) (layers F.Cu F.Paste F.Mask)
       (net 1 Earth))
     (model ${KISYS3DMOD}/Connector_USB.3dshapes/USB_C_Plug_Molex_105444.wrl
@@
   (segment (start 147.46 91.5) (end 148.25 91.5) (width 0.2) (layer F.Cu) (net 1))
   (segment (start 146 90.04) (end 147.46 91.5) (width 0.2) (layer F.Cu) (net 1))
-  (via (at 146.67 90.88) (size 0.8) (drill 0.4) (layers F.Cu B.Cu) (net 1))
   (segment (start 145.98 91.57) (end 146.67 90.88) (width 0.3) (layer F.Cu) (net 1))
   (segment (start 145.98 98.75) (end 145.98 91.57) (width 0.3) (layer F.Cu) (net 1))
@@
   (segment (start 142.5 92.463998) (end 140.26 94.703998) (width 0.2) (layer F.Cu) (net 4))
   (segment (start 142.5 90.04) (end 142.5 92.463998) (width 0.2) (layer F.Cu) (net 4))
-  (via (at 142.75 93.25) (size 0.8) (drill 0.4) (layers F.Cu B.Cu) (net 14))
   (segment (start 142.455 100.865) (end 142.865 101.275) (width 0.2) (layer F.Cu) (net 13))
   (segment (start 143.475 98.0932) (end 142.455 99.1132) (width 0.2) (layer F.Cu) (net 13))
@@
   (segment (start 143 92.409301) (end 143.475 92.884301) (width 0.2) (layer F.Cu) (net 13))
   (segment (start 143 90.04) (end 143 92.409301) (width 0.2) (layer F.Cu) (net 13))
+  (via (at 142.75 93.25) (size 0.8) (drill 0.4) (layers F.Cu B.Cu) (net 14))
   (segment (start 142.005 100.865) (end 142.005 98.9268) (width 0.2) (layer F.Cu) (net 14))
   (segment (start 141.595 101.275) (end 142.005 100.865) (width 0.2) (layer F.Cu) (net 14))

Commit message: Added new files
Parts:
- P1: value USB_C_Plug_USB2.0 -> 105444-0001
- moved H1 0.25 mm to (131.9, 110.0)
- moved H2 0.20 mm to (154.6, 110.0)
Connections:
- U1 pad 1: Net-(U1-Pad1) -> Earth
Changed lines of the file:
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@@
     (zones 0)
     (modules 14)
-    (nets 23)
+    (nets 22)
   )
   (page A4)
@@
     (47 F.CrtYd user)
     (48 B.Fab user)
-    (49 F.Fab user hide)
+    (49 F.Fab user)
   )
   (setup
@@
       (drillshape 0)
       (scaleselection 1)
-      (outputdirectory "C:/Users/Josh/Documents/ExpansionCards-main/Design Files/Complete Design Files/USB-C to TTL UART/Gerbers/"))
+      (outputdirectory "C:/Users/Josh/Documents/ExpansionCards-main/Design Files/Production Files/USB-C to UART versions/USB-C to UART  Production/Gerbers/"))
   )
   (net 0 "")
@@
   (net 20 5V)
   (net 21 "Net-(C2-Pad1)")
-  (net 22 "Net-(U1-Pad1)")
   (net_class Default "This is the default net class."
     (clearance 0.2)
@@
     (add_net "Net-(P1-PadA5)")
     (add_net "Net-(P1-PadB5)")
-    (add_net "Net-(U1-Pad1)")
     (add_net "Net-(U1-Pad10)")
     (add_net "Net-(U1-Pad11)")
@@
   )
   (module MountingHole:MountingHole_2.2mm_M2 (layer F.Cu)
-    (at 154.75 110)
+    (at 154.55 110)
     (descr "Mounting Hole 2.2mm, no annular, M2")
     (tags "mounting hole 2.2mm no annular m2")
@@
   )
   (module MountingHole:MountingHole_2.2mm_M2 (layer F.Cu)
-    (at 131.7 110)
+    (at 131.95 110)
     (descr "Mounting Hole 2.2mm, no annular, M2")
     (tags "mounting hole 2.2mm no annular m2")
@@
       (effects (font (size 1 1) (thickness 0.15)))
     )
-    (fp_text value 1uF (at 0 1.16) (layer F.Fab)
+    (fp_text value 1uF (at -4.7 0) (layer F.SilkS)
       (effects (font (size 1 1) (thickness 0.15)))
     )
@@
       (effects (font (size 1 1) (thickness 0.15)))
     )
-    (fp_text value 1uF (at 0 1.16) (layer F.Fab)
+    (fp_text value 1uF (at 0.07 2.74) (layer F.SilkS)
       (effects (font (size 1 1) (thickness 0.15)))
     )
@@
       (effects (font (size 1 1) (thickness 0.15)))
     )
-    (fp_text value AP2112K-3.3 (at 0 2.9 90) (layer F.Fab)
-      (effects (font (size 1 1) (thickness 0.15)))
+    (fp_text value AP2112K-3.3 (at 0.09 -4.04 270) (layer F.SilkS)
+      (effects (font (size 0.5 0.5) (thickness 0.125)))
     )
     (fp_line (start -0.9 1.61) (end 0.9 1.61) (layer F.SilkS) (width 0.12))
@@
       (effects (font (size 1 1) (thickness 0.15)))
     )
-    (fp_text value 5.1k (at 0 1.17) (layer F.Fab)
+    (fp_text value 5.1k (at -2.55 0) (layer F.SilkS)
       (effects (font (size 1 1) (thickness 0.15)))
     )
@@
       (effects (font (size 1 1) (thickness 0.15)))
     )
-    (fp_text value 0.1uF (at 0 1.16) (layer F.Fab)
+    (fp_text value 0.1uF (at -5.1 0.15) (layer F.SilkS)
       (effects (font (size 1 1) (thickness 0.15)))
     )
@@
       (effects (font (size 1 1) (thickness 0.15)))
     )
-    (fp_text value 10nF (at 0 1.16) (layer F.Fab)
+    (fp_text value 10nF (at 2.9 -0.15) (layer F.SilkS)
       (effects (font (size 1 1) (thickness 0.15)))
     )
@@
       (effects (font (size 1 1) (thickness 0.15)))
     )
-    (fp_text value USB_C_Plug_USB2.0 (at 0 -1.96) (layer F.Fab)
+    (fp_text value 105444-0001 (at 4.75 4.6) (layer F.SilkS)
       (effects (font (size 1 1) (thickness 0.15)))
     )
@@
       (effects (font (size 1 1) (thickness 0.15)))
     )
-    (fp_text value CH340C (at 0 5.9 90) (layer F.Fab)
+    (fp_text value CH340C (at 0 -7.3 90) (layer F.SilkS)
       (effects (font (size 1 1) (thickness 0.15)))
     )
@@
     )
     (pad 1 smd roundrect (at -2.475 -4.445 270) (size 1.95 0.6) (layers F.Cu F.Paste F.Mask) (roundrect_rratio 0.25)
-      (net 22 "Net-(U1-Pad1)"))
+      (net 1 Earth))
     (pad 2 smd roundrect (at -2.475 -3.175 270) (size 1.95 0.6) (layers F.Cu F.Paste F.Mask) (roundrect_rratio 0.25)
       (net 18 TXO))
