File: Hardware/USB-C to TLL UART.sch (KiCad schematic (older format))
At the start: 11 parts, among them IC1 74LVC1G08SE-7, J1 Conn_01x06_Female, P1 USB_C_Plug_USB2.0, U1 CH340C, U2 AP2112K-3.3

Commit message: Updated Files
Parts:
- removed IC1: 74LVC1G08SE-7, SamacSys_Parts:SOT65P210X110-5N, symbol SamacSys_Parts:74LVC1G08SE-7
- C1: value 10nF -> 0.1uF
- C2: value 100nF -> 10nF
- P1: footprint SnapEDA Library:GCT_USB4155-03-C_REVA -> Expansion_Card:USB_C_Plug_Molex_105444
Connections:
- net 5V: now also C1.1
- net Earth: no longer U1.1 (GND)
- net VCC: no longer C2.1
- net at U1.4 (V3): now also C2.1; no longer C1.1
- no-connect marks 9 -> 6

Commit message: Added new files
Connections:
- net Earth: now also U1.1 (GND)
Changed lines of the file:
@@
 Text GLabel 4800 1900 1    50   Input ~ 0
 VCC
+$Comp
+L power:Earth #PWR05
+U 1 1 62B11BDF
+P 4800 3100
+F 0 "#PWR05" H 4800 2850 50  0001 C CNN
+F 1 "Earth" H 4800 2950 50  0001 C CNN
+F 2 "" H 4800 3100 50  0001 C CNN
+F 3 "~" H 4800 3100 50  0001 C CNN
+	1    4800 3100
+	1    0    0    -1
+$EndComp
 $EndSCHEMATC
